File: Hardware/JBC controller.kicad_pcb (KiCad board)
At the start: 2 copper layers, 70 x 50 mm, 42 parts, among them J1 Conn_01x04_Male, J2 XT30, J3 Conn_01x04_Male, J4 Conn_01x01_Male, J5 Conn_01x04_Male, J6 Conn_01x05_Male, J7 Conn_01x01_Male, Q1 BC846, Q2 SI4101DY, SW1 JS202011AQN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

Commit message: Hardware v0.1
Other:
- board text added: "rcoleman.uk JBC controller v0.2"
- board text removed: "rcoleman.uk JBC controller v0.1"
